File: control_logic.kicad_sch (KiCad schematic)
At the start: 59 parts, among them J12 SWD Header, J17 TC2050, SW1 KMR721NGLFS, SW2 KMR721NGLFS, U10 L7805, U11 MCP2562-E-SN, U12 STM32F105RCTx, U13 AZ1117I-3.3, U15 TPD4E1U06, Y3 8MHz 12pF

Commit message: added balancer thermistor info; changed MCU pinout to support CAN bootloading
Parts:
- added C39: 100n, symbol Device:C
Connections:
- net +5V: now also C39.1
- net CAN_RX: now also U12.57 (PB5); no longer U12.61 (PB8)
- net CAN_TX: now also U12.58 (PB6); no longer U12.62 (PB9)
- net CHRG_IND_LED_4: now also U12.28 (PB2); no longer U12.57 (PB5)
- net GND: now also C39.2
- net I2C1_SCL: now also U12.61 (PB8); no longer U12.58 (PB6)
- no-connect marks 24 -> 23
Other:
- note added: "INFO: those pins support CAN bootloader"
- note removed: "todo: add can bootloader"
- note removed: "todo: add can bootloader (AN3154)"
Changed lines of the file:
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@@
 		)
 	)
+	(text "INFO: those pins support CAN bootloader"
+		(exclude_from_sim no)
+		(at 382.27 103.124 0)
+		(effects
+			(font
+				(size 1.27 1.27)
+			)
+		)
+	)
 	(text "controller"
 		(exclude_from_sim no)
@@
 		)
 	)
-	(text "todo: add can bootloader"
-		(exclude_from_sim no)
-		(at 44.45 130.048 0)
-		(effects
-			(font
-				(size 1.27 1.27)
-			)
-		)
-	)
 	(text "programming adapters"
 		(exclude_from_sim no)
@@
 		)
 	)
-	(text "todo: add can bootloader (AN3154)"
-		(exclude_from_sim no)
-		(at 381 110.998 0)
-		(effects
-			(font
-				(size 1.27 1.27)
-			)
-		)
-	)
 	(text "active low (power good)"
 		(exclude_from_sim no)
@@
 	)
 	(no_connect
-		(at 350.52 93.98)
-	)
-	(no_connect
 		(at 350.52 60.96)
 	)
@@
 	(wire
 		(pts
-			(xy 353.06 109.22) (xy 350.52 109.22)
+			(xy 351.79 109.22) (xy 350.52 109.22)
 		)
 		(stroke
@@
 	(wire
 		(pts
+			(xy 350.52 93.98) (xy 351.79 93.98)
+		)
+		(stroke
+			(width 0)
+			(type default)
+		)
+	)
+	(wire
+		(pts
 			(xy 53.34 114.3) (xy 53.34 113.03)
 		)
@@
 		)
 	)
-	(global_label "CAN_RX"
+	(global_label "CHRG_IND_LED_4"
 		(shape input)
-		(at 353.06 109.22 0)
+		(at 351.79 93.98 0)
 		(fields_autoplaced yes)
 		(effects
@@
 		)
 		(property "Intersheetrefs" "${INTERSHEET_REFS}"
-			(at 363.1814 109.22 0)
+			(at 370.6804 93.98 0)
 			(effects
 				(font
@@
 		)
 	)
-	(global_label "CHRG_IND_LED_3"
+	(global_label "CAN_RX"
 		(shape input)
-		(at 326.39 220.98 0)
+		(at 351.79 101.6 0)
 		(fields_autoplaced yes)
 		(effects
@@
 		)
 		(property "Intersheetrefs" "${INTERSHEET_REFS}"
-			(at 345.2804 220.98 0)
+			(at 361.9114 101.6 0)
 			(effects
 				(font
@@
 		)
 	)
-	(global_label "CAN_TX"
+	(global_label "CHRG_IND_LED_3"
 		(shape input)
-		(at 353.06 111.76 0)
+		(at 326.39 220.98 0)
 		(fields_autoplaced yes)
 		(effects
@@
 		)
 		(property "Intersheetrefs" "${INTERSHEET_REFS}"
-			(at 362.879 111.76 0)
+			(at 345.2804 220.98 0)
 			(effects
 				(font
@@
 	(global_label "I2C1_SCL"
 		(shape input)
-		(at 351.79 104.14 0)
+		(at 351.79 109.22 0)
 		(fields_autoplaced yes)
 		(effects
@@
 		)
 		(property "Intersheetrefs" "${INTERSHEET_REFS}"
-			(at 363.5442 104.14 0)
+			(at 363.5442 109.22 0)
 			(effects
 				(font
@@
 		)
 	)
-	(global_label "CHRG_IND_LED_4"
-		(shape input)
-		(at 351.79 101.6 0)
-		(fields_autoplaced yes)
-		(effects
-			(font
-				(size 1.27 1.27)
-			)
-			(justify left)
-		)
-		(property "Intersheetrefs" "${INTERSHEET_REFS}"
-			(at 370.6804 101.6 0)
-			(effects
-				(font
-					(size 1.27 1.27)
-				)
-				(justify left)
-				(hide yes)
-			)
-		)
-	)
 	(global_label "BOOT"
 		(shape input)
@@
 		)
 	)
+	(global_label "CAN_TX"
+		(shape input)
+		(at 351.79 104.14 0)
+		(fields_autoplaced yes)
+		(effects
+			(font
+				(size 1.27 1.27)
+			)
+			(justify left)
+		)
+		(property "Intersheetrefs" "${INTERSHEET_REFS}"
+			(at 361.609 104.14 0)
+			(effects
+				(font
+					(size 1.27 1.27)
+				)
+				(justify left)
+				(hide yes)
+			)
+		)
+	)
 	(hierarchical_label "I2C2_SCL"
 		(shape bidirectional)
@@
 	)
 	(symbol
+		(lib_name "GND_1")
+		(lib_id "power:GND")
+		(at 76.2 63.5 0)
+		(unit 1)
+		(exclude_from_sim no)
+		(in_bom yes)
+		(on_board yes)
+		(dnp no)
+		(fields_autoplaced yes)
+		(property "Reference" "#PWR073"
+			(at 76.2 69.85 0)
+			(effects
+				(font
+					(size 1.27 1.27)
+				)
+				(hide yes)
+			)
+		)
+		(property "Value" "GND"
+			(at 76.2 68.58 0)
+			(effects
+				(font
+					(size 1.27 1.27)
+				)
+			)
+		)
+		(property "Footprint" ""
+			(at 76.2 63.5 0)
+			(effects
+				(font
+					(size 1.27 1.27)
+				)
+				(hide yes)
+			)
+		)
+		(property "Datasheet" ""
+			(at 76.2 63.5 0)
+			(effects
+				(font
+					(size 1.27 1.27)
+				)
+				(hide yes)
+			)
+		)
+		(property "Description" "Power symbol creates a global label with name \"GND\" , ground"
+			(at 76.2 63.5 0)
+			(effects
+				(font
+					(size 1.27 1.27)
+				)
+				(hide yes)
+			)
+		)
+		(pin "1"
+		)
+		(instances
+			(project "rapid_power_module"
+				(path "/afc8cbd3-9ea8-40a2-afae-ed6bd0fe7e6e/5220dff6-c057-4538-a5b2-0b6e4cf779ce"
+					(reference "#PWR073")
+					(unit 1)
+				)
+			)
+		)
+	)
+	(symbol
 		(lib_id "power:GND")
 		(at 69.85 200.66 0)
@@
 	)
 	(symbol
+		(lib_id "Device:C")
+		(at 76.2 59.69 0)
+		(unit 1)
+		(exclude_from_sim no)
+		(in_bom yes)
+		(on_board yes)
+		(dnp no)
+		(fields_autoplaced yes)
+		(property "Reference" "C39"
+			(at 80.01 58.4199 0)
+			(effects
+				(font
+					(size 1.27 1.27)
+				)
+				(justify left)
+			)
+		)
+		(property "Value" "100n"
+			(at 80.01 60.9599 0)
+			(effects
+				(font
+					(size 1.27 1.27)
+				)
+				(justify left)
+			)
+		)
+		(property "Footprint" ""
+			(at 77.1652 63.5 0)
+			(effects
+				(font
+					(size 1.27 1.27)
+				)
+				(hide yes)
+			)
+		)
+		(property "Datasheet" "~"
+			(at 76.2 59.69 0)
+			(effects
+				(font
+					(size 1.27 1.27)
+				)
+				(hide yes)
+			)
+		)
+		(property "Description" "Unpolarized capacitor"
+			(at 76.2 59.69 0)
+			(effects
+				(font
+					(size 1.27 1.27)
+				)
+				(hide yes)
+			)
+		)
+		(pin "1"
+		)
+		(pin "2"
+		)
+		(instances
+			(project ""
+				(path "/afc8cbd3-9ea8-40a2-afae-ed6bd0fe7e6e/5220dff6-c057-4538-a5b2-0b6e4cf779ce"
+					(reference "C39")
+					(unit 1)
+				)
+			)
+		)
+	)
+	(symbol
 		(lib_name "GND_1")
 		(lib_id "power:GND")
@@
 					(unit 1)
 				)
+			)
+		)
+	)
+	(symbol
+		(lib_id "power:+5V")
+		(at 76.2 55.88 0)
+		(unit 1)
+		(exclude_from_sim no)
+		(in_bom yes)
+		(on_board yes)
+		(dnp no)
+		(property "Reference" "#PWR069"
+			(at 76.2 59.69 0)
+			(effects
+				(font
+					(size 1.27 1.27)
+				)
+				(hide yes)
+			)
+		)
+		(property "Value" "+5V"
+			(at 75.946 52.324 0)
+			(effects
+				(font
+					(size 1.27 1.27)
+				)
+			)
+		)
+		(property "Footprint" ""
+			(at 76.2 55.88 0)
+			(effects
+				(font
+					(size 1.27 1.27)
+				)
+				(hide yes)
+			)
+		)
+		(property "Datasheet" ""
+			(at 76.2 55.88 0)
+			(effects
+				(font
+					(size 1.27 1.27)
+				)
+				(hide yes)
+			)
+		)
+		(property "Description" "Power symbol creates a global label with name \"+5V\""
+			(at 76.2 55.88 0)
+			(effects
+				(font
+					(size 1.27 1.27)
+				)
+				(hide yes)
+			)
+		)
+		(pin "1"
+		)
+		(instances
+			(project "rapid_power_module"
+				(path "/afc8cbd3-9ea8-40a2-afae-ed6bd0fe7e6e/5220dff6-c057-4538-a5b2-0b6e4cf779ce"
+					(reference "#PWR069")
+					(unit 1)
+				)

Commit message: Changed Balancer layout to support OVP, UVP and UVP-circumvention; added UVP-circumvention arming connector
Connections:
- net BAL_ALERT: no longer names the net of U12.24 (PC4)
- net I2C2_SCL: no longer names the net of U12.29 (PB10)
- net I2C2_SDA: no longer names the net of U12.30 (PB11)
- net RST_SHUT: no longer names the net of U12.2 (PC13)
- net TS2: no longer names the net of U12.17 (PA3)
- no-connect marks 23 -> 26
Other:
- note added: "todo: -ensure 5v -why are we connecting 3v3 and not nrst? -shouldnt we also protect BOOT?"
- note removed: "int from 25 to 51 PG from 39 to 36 REGIN und BREG verbunden mit STM32"
- note removed: "mv 16 -> 2"
- note removed: "todo: -ensure 5v -why are we connecting 3v3 and not nrst? -add a second i2c-swd-header (one for charger) -shouldnt we also protect BOOT?"
Changed lines of the file:
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@@
 		)
 	)
-	(text "mv 16 -> 2"
-		(exclude_from_sim no)
-		(at 359.41 48.26 0)
-		(effects
-			(font
-				(size 1.27 1.27)
-			)
-		)
-	)
 	(text "\"connect INT, STAT1, STAT2 and PG \nto a logic rail via 10k resistor\" \n-> (bq25750 man. page 5)"
 		(exclude_from_sim no)
@@
 		)
 	)
-	(text "todo: \n-ensure 5v\n-why are we connecting 3v3 and not nrst?\n-add a second i2c-swd-header \n(one for charger)\n-shouldnt we also protect BOOT?"
+	(text "todo: \n-ensure 5v\n-why are we connecting 3v3 and not nrst?\n-shouldnt we also protect BOOT?"
 		(exclude_from_sim no)
 		(at 64.008 80.264 0)
@@
 		)
 	)
-	(text "int from 25 to 51\nPG from 39 to 36\nREGIN und BREG verbunden mit STM32"
-		(exclude_from_sim no)
-		(at 296.418 110.998 0)
-		(effects
-			(font
-				(size 1.27 1.27)
-			)
-		)
-	)
 	(text "charging done"
 		(exclude_from_sim no)
@@
 	)
 	(no_connect
+		(at 350.52 53.34)
+	)
+	(no_connect
 		(at 350.52 73.66)
 	)
@@
 	)
 	(no_connect
+		(at 314.96 76.2)
+	)
+	(no_connect
 		(at 350.52 60.96)
 	)
@@
 		(at 350.52 66.04)
 	)
+	(no_connect
+		(at 314.96 99.06)
+	)
 	(wire
 		(pts
@@
 	(wire
 		(pts
-			(xy 350.52 114.3) (xy 353.06 114.3)
-		)
-		(stroke
-			(width 0)
-			(type default)
-		)
-	)
-	(wire
-		(pts
 			(xy 287.02 35.56) (xy 298.45 35.56)
 		)
@@
 	(wire
 		(pts
-			(xy 350.52 116.84) (xy 353.06 116.84)
-		)
-		(stroke
-			(width 0)
-			(type default)
-		)
-	)
-	(wire
-		(pts
 			(xy 384.81 222.25) (xy 384.81 220.98)
 		)
@@
 	(wire
 		(pts
-			(xy 353.06 53.34) (xy 350.52 53.34)
-		)
-		(stroke
-			(width 0)
-			(type default)
-		)
-	)
-	(wire
-		(pts
 			(xy 26.67 215.9) (xy 26.67 218.44)
 		)
@@
 	(wire
 		(pts
-			(xy 313.69 99.06) (xy 314.96 99.06)
-		)
-		(stroke
-			(width 0)
-			(type default)
-		)
-	)
-	(wire
-		(pts
 			(xy 358.14 25.4) (xy 346.71 25.4)
 		)
@@
 	(wire
 		(pts
-			(xy 353.06 111.76) (xy 350.52 111.76)
-		)
-		(stroke
-			(width 0)
-			(type default)
-		)
-	)
-	(wire
-		(pts
 			(xy 337.82 38.1) (xy 337.82 35.56)
 		)
@@
 		)
 	)
-	(hierarchical_label "I2C2_SCL"
-		(shape bidirectional)
-		(at 353.06 114.3 0)
-		(effects
-			(font
-				(size 1.27 1.27)
-			)
-			(justify left)
-		)
-	)
 	(hierarchical_label "CAN+"
 		(shape input)
@@
 		)
 	)
-	(hierarchical_label "RST_SHUT"
-		(shape output)
-		(at 313.69 99.06 180)
-		(effects
-			(font
-				(size 1.27 1.27)
-			)
-			(justify right)
-		)
-	)
 	(hierarchical_label "main_voltage"
 		(shape input)
@@
 		)
 	)
-	(hierarchical_label "I2C2_SDA"
-		(shape bidirectional)
-		(at 353.06 116.84 0)
-		(effects
-			(font
-				(size 1.27 1.27)
-			)
-			(justify left)
-		)
-	)
-	(hierarchical_label "BAL_ALERT"
-		(shape input)
-		(at 314.96 76.2 180)
-		(effects
-			(font
-				(size 1.27 1.27)
-			)
-			(justify right)
-		)
-	)
 	(hierarchical_label "CE_N"
 		(shape output)
@@
 		(effects
 			(font
-				(size 1.27 1.27)
-			)
-			(justify left)
-		)
-	)
-	(hierarchical_label "TS2"
-		(shape input)
-		(at 353.06 53.34 0)
-		(effects
-			(font

Commit message: added explanations for balancer schematic and some component values
Other:
- note removed: "todo: -ensure 5v -why are we connecting 3v3 and not nrst? -shouldnt we also protect BOOT?"
Changed lines of the file:
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@@
 	(rectangle
 		(start 13.97 13.97)
-		(end 107.95 123.19)
+		(end 90.17 123.19)
 		(stroke
 			(width 0)
@@
 			)
 			(justify left)
-		)
-	)
-	(text "todo: \n-ensure 5v\n-why are we connecting 3v3 and not nrst?\n-shouldnt we also protect BOOT?"
-		(exclude_from_sim no)
-		(at 64.008 80.264 0)
-		(effects
-			(font
-				(size 1.27 1.27)
-			)
-			(justify left)
