File: control_logic.kicad_sch (KiCad schematic)
At the start: 71 parts, among them J12 SWD Header, J17 TC2050, SW1 TS342A2P, SW2 TS342A2P, U1 INA181A1, U10 L7805, U11 MCP2562-E-SN, U12 STM32F105RCTx, U13 AZ1117I-3.3, U15 TPD4E1U06, Y3 8MHz 12pF

Commit message: added current sensing circuit
Parts:
- removed C1: 100n, Capacitor_SMD:C_0402_1005Metric, symbol Device:C
- removed D13, D14: D, Diode_SMD:D_SOD-123F, symbol Device:D
- removed F?: 10A, Fuse:Fuse_1206_3216Metric, symbol Device:Fuse_Small
- removed R1: 25m, Resistor_SMD:R_1206_3216Metric_Pad1.30x1.75mm_HandSolder, symbol Device:R
- removed U1: INA181A1, Package_TO_SOT_SMD:SOT-23-6, symbol Amplifier_Current:INA181
Other:
- note added: "from batteries"
- note added: "redundand but does not hurt"
- moved on the sheet: R17, R4

Commit message: finished adding sensing-capabilities (incl. routing)
Parts:
- removed R17, R4: R, symbol Device:R
Connections:
- net sense_V_bat: no longer names the net of U12.15 (PA1)
- no-connect marks 29 -> 30
Other:
- note removed: "ADC12_IN1"

Commit message: preparing for order
Parts:
- added TP_3V3, TP_5V, TP_CAN_RX, TP_CAN_TX, TP_I2C_SCL, TP_I2C_SDA, TP_SWCLK, TP_SWDIO, TP_SWO: TestPoint, symbol Connector:TestPoint
- J17: now not fitted
Connections:
- net +3V3: now also TP_3V3.1
- net +5V: now also TP_5V.1
- net CAN_RX: now also TP_CAN_RX.1
- net CAN_TX: now also TP_CAN_TX.1
- net CHRG_IND_LED_2: now also U12.50 (PA15); no longer U12.55 (PB3)
- net I2C1_SCL: now also TP_I2C_SCL.1
- net I2C1_SDA: now also TP_I2C_SDA.1
- net SWCLK: now also TP_SWCLK.1
- net SWDIO: now also TP_SWDIO.1
- net SWO: now also U12.55 (PB3), TP_SWO.1; no longer U12.50 (PA15)
Other:
- moved on the sheet: C15, C63, J12, R35, R66, R67, R77, R78, R86, R87, R88, R92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

Commit message: added test points
Parts:
- TP10: renamed from TP_SWO; footprint (none) -> TestPoint:TestPoint_Pad_D2.0mm
- TP11: renamed from TP_CAN_RX; footprint (none) -> TestPoint:TestPoint_Pad_D2.0mm
- TP12: renamed from TP_3V3; footprint (none) -> TestPoint:TestPoint_Pad_D2.0mm
- TP13: renamed from TP_SWCLK; footprint (none) -> TestPoint:TestPoint_Pad_D2.0mm
- TP5: renamed from TP_5V; footprint (none) -> TestPoint:TestPoint_Pad_D2.0mm
- TP6: renamed from TP_SWDIO; footprint (none) -> TestPoint:TestPoint_Pad_D2.0mm
- TP7: renamed from TP_I2C_SCL; footprint (none) -> TestPoint:TestPoint_Pad_D2.0mm
- TP8: renamed from TP_I2C_SDA; footprint (none) -> TestPoint:TestPoint_Pad_D2.0mm
- TP9: renamed from TP_CAN_TX; footprint (none) -> TestPoint:TestPoint_Pad_D2.0mm
Changed lines of the file:
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@@
 	(wire
 		(pts
-			(xy 25.4 38.1) (xy 25.4 62.23)
+			(xy 24.13 38.1) (xy 24.13 62.23)
 		)
 		(stroke
@@
 	(wire
 		(pts
-			(xy 25.4 38.1) (xy 38.1 38.1)
+			(xy 24.13 38.1) (xy 38.1 38.1)
 		)
 		(stroke
@@
 	(wire
 		(pts
-			(xy 25.4 62.23) (xy 39.37 62.23)
+			(xy 24.13 62.23) (xy 39.37 62.23)
 		)
 		(stroke
@@
 		(on_board yes)
 		(dnp no)
-		(property "Reference" "TP_3V3"
+		(property "Reference" "TP12"
 			(at 63.5 214.6299 90)
 			(effects
@@
 			)
 		)
-		(property "Footprint" ""
+		(property "Footprint" "TestPoint:TestPoint_Pad_D2.0mm"
 			(at 58.42 220.98 0)
 			(effects
@@
 			(project "rapid_power_module"
 				(path "/afc8cbd3-9ea8-40a2-afae-ed6bd0fe7e6e/5220dff6-c057-4538-a5b2-0b6e4cf779ce"
-					(reference "TP_3V3")
+					(reference "TP12")
 					(unit 1)
 				)
@@
 		(dnp no)
 		(fields_autoplaced yes)
-		(property "Reference" "TP_CAN_TX"
+		(property "Reference" "TP9"
 			(at 33.02 137.6679 0)
 			(effects
@@
 			)
 		)
-		(property "Footprint" ""
+		(property "Footprint" "TestPoint:TestPoint_Pad_D2.0mm"
 			(at 35.56 142.24 0)
 			(effects
@@
 			(project "rapid_power_module"
 				(path "/afc8cbd3-9ea8-40a2-afae-ed6bd0fe7e6e/5220dff6-c057-4538-a5b2-0b6e4cf779ce"
-					(reference "TP_CAN_TX")
+					(reference "TP9")
 					(unit 1)
 				)
@@
 		(on_board yes)
 		(dnp no)
-		(property "Reference" "TP_CAN_RX"
+		(property "Reference" "TP11"
 			(at 36.322 146.304 0)
 			(effects
@@
 			)
 		)
-		(property "Footprint" ""
+		(property "Footprint" "TestPoint:TestPoint_Pad_D2.0mm"
 			(at 41.91 144.78 0)
 			(effects
@@
 			(project "rapid_power_module"
 				(path "/afc8cbd3-9ea8-40a2-afae-ed6bd0fe7e6e/5220dff6-c057-4538-a5b2-0b6e4cf779ce"
-					(reference "TP_CAN_RX")
+					(reference "TP11")
 					(unit 1)
 				)
@@
 		(on_board yes)
 		(dnp no)
-		(property "Reference" "TP_SWDIO"
+		(property "Reference" "TP6"
 			(at 24.13 36.3219 0)
 			(effects
@@
 			)
 		)
-		(property "Footprint" ""
+		(property "Footprint" "TestPoint:TestPoint_Pad_D2.0mm"
 			(at 31.75 34.29 0)
 			(effects
@@
 			(project "rapid_power_module"
 				(path "/afc8cbd3-9ea8-40a2-afae-ed6bd0fe7e6e/5220dff6-c057-4538-a5b2-0b6e4cf779ce"
-					(reference "TP_SWDIO")
+					(reference "TP6")
 					(unit 1)
 				)
@@
 		(on_board yes)
 		(dnp no)
-		(property "Reference" "TP_5V"
+		(property "Reference" "TP5"
 			(at 20.828 210.82 90)
 			(effects
@@
 			)
 		)
-		(property "Footprint" ""
+		(property "Footprint" "TestPoint:TestPoint_Pad_D2.0mm"
 			(at 24.13 210.82 0)
 			(effects
@@
 			(project "rapid_power_module"
 				(path "/afc8cbd3-9ea8-40a2-afae-ed6bd0fe7e6e/5220dff6-c057-4538-a5b2-0b6e4cf779ce"
-					(reference "TP_5V")
+					(reference "TP5")
 					(unit 1)
 				)
@@
 		(on_board yes)
 		(dnp no)
-		(property "Reference" "TP_SWO"
+		(property "Reference" "TP10"
 			(at 34.544 42.672 0)
 			(effects
@@
 			)
 		)
-		(property "Footprint" ""
+		(property "Footprint" "TestPoint:TestPoint_Pad_D2.0mm"
 			(at 40.64 40.64 0)
 			(effects
@@
 			(project "rapid_power_module"
 				(path "/afc8cbd3-9ea8-40a2-afae-ed6bd0fe7e6e/5220dff6-c057-4538-a5b2-0b6e4cf779ce"
-					(reference "TP_SWO")
+					(reference "TP10")
 					(unit 1)
 				)
@@
 		(dnp no)
 		(fields_autoplaced yes)
-		(property "Reference" "TP_SWCLK"
+		(property "Reference" "TP13"
 			(at 77.47 36.0679 0)
 			(effects
@@
 			)
 		)
-		(property "Footprint" ""
+		(property "Footprint" "TestPoint:TestPoint_Pad_D2.0mm"
 			(at 80.01 40.64 0)
 			(effects
@@
 			(project "rapid_power_module"
 				(path "/afc8cbd3-9ea8-40a2-afae-ed6bd0fe7e6e/5220dff6-c057-4538-a5b2-0b6e4cf779ce"
-					(reference "TP_SWCLK")
+					(reference "TP13")
 					(unit 1)
 				)
@@
 		(dnp no)
 		(fields_autoplaced yes)
-		(property "Reference" "TP_I2C_SCL"
+		(property "Reference" "TP7"
 			(at 33.02 103.3779 0)
 			(effects
@@
 			)
 		)
-		(property "Footprint" ""
+		(property "Footprint" "TestPoint:TestPoint_Pad_D2.0mm"
 			(at 35.56 107.95 0)
 			(effects
@@
 			(project "rapid_power_module"
 				(path "/afc8cbd3-9ea8-40a2-afae-ed6bd0fe7e6e/5220dff6-c057-4538-a5b2-0b6e4cf779ce"
-					(reference "TP_I2C_SCL")
+					(reference "TP7")
 					(unit 1)
 				)
@@
 		(dnp no)
 		(fields_autoplaced yes)
-		(property "Reference" "TP_I2C_SDA"
+		(property "Reference" "TP8"
 			(at 33.02 112.5219 0)
 			(effects
@@
 			)
 		)
-		(property "Footprint" ""
+		(property "Footprint" "TestPoint:TestPoint_Pad_D2.0mm"
 			(at 25.4 110.49 0)
 			(effects
@@
 			(project "rapid_power_module"
 				(path "/afc8cbd3-9ea8-40a2-afae-ed6bd0fe7e6e/5220dff6-c057-4538-a5b2-0b6e4cf779ce"
-					(reference "TP_I2C_SDA")
+					(reference "TP8")
 					(unit 1)
 				)

Commit message: fix silkscreen issues and start implementing small layout improvements, cleanup repo
Parts:
- D10, D8: value ~ -> (none)

Commit message: finished routing adaptions
Parts:
- removed R9: 10k, Resistor_SMD:R_0402_1005Metric, symbol Device:R
- renumbered C15 to C10, C61 to C11, C80 to C12, C58 to C13, C60 to C14, C63 to C15, C79 to C16, C67 to C17, C68 to C18, C69 to C19, C70 to C20, C71 to C21, C72 to C22, C73 to C23, C74 to C24, C77 to C25, C75 to C26, C76 to C27, C78 to C28, D4 to D10, D5 to D11, D6 to D12, D8 to D4, D10 to D5, D17 to D6, D18 to D7, D19 to D8, D3 to D9, J17 to J8, J12 to J9, R92 to R1, R18 to R10, R19 to R11, R20 to R12, R21 to R13, R34 to R14, R76 to R15, R26 to R16, R10 to R17, R11 to R18, R12 to R19, R86 to R2, R13 to R20, R14 to R21, R15 to R22, R74 to R23, R87 to R3, R67 to R4, R66 to R5, R77 to R6, R78 to R7, R35 to R8, R88 to R9, U13 to U1, U15 to U2, U11 to U3, U10 to U4, U12 to U5, Y3 to Y1
Connections:
- net +3V3: no longer U2.5 (IO4)
- net at J8.1 (Pin_1), R1.2: now also U2.5 (IO4)

Commit message: last changes (components) for ordering
Parts:
- C17: LCSC C368809 -> C23733; Manufacturer Samsung Electro-Mechanics -> (none)
- C23, C27: LCSC C60133 -> C15195; Manufacturer YAGEO -> (none)
- C25, C28: LCSC C76946 -> C32949; Manufacturer Murata Electronics -> (none)
- R1, R2, R3, R9: value 22 -> 22R
- SW1, SW2: value TS342A2P -> (none); footprint Button_Switch_SMD:SW_Push_SPST_NO_Alps_SKRK -> Button_Switch_SMD:SW_SPST_TS-1088-xR020; LCSC C5373431 -> C720477
Changed lines of the file:
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@@
 			)
 		)
-		(property "Datasheet" "https://www.lcsc.com/datasheet/lcsc_datasheet_2304140030_YAGEO-CC0402KRX7R9BB103_C60133.pdf"
+		(property "Datasheet" ""
 			(at 346.71 30.48 0)
 			(hide yes)
@@
 			)
 		)
-		(property "Description" "50V 10nF X7R ±10% 0402 Multilayer Ceramic Capacitors MLCC - SMD/SMT ROHS"
+		(property "Description" ""
 			(at 346.71 30.48 0)
 			(hide yes)
@@
 			)
 		)
-		(property "LCSC" "C60133"
+		(property "LCSC" "C15195"
 			(at 346.71 30.48 0)
 			(hide yes)
@@
 			)
 		)
-		(property "Manufacturer" "YAGEO"
+		(property "Manufacturer" ""
 			(at 346.71 30.48 0)
 			(hide yes)
@@
 			)
 		)
-		(property "Datasheet" "https://www.lcsc.com/datasheet/lcsc_datasheet_2304140030_Samsung-Electro-Mechanics-CL05A475KP5NRNC_C368809.pdf"
-			(at 265.43 30.48 0)
-			(hide yes)
-			(show_name no)
-			(do_not_autoplace no)
-			(effects
-				(font
-					(size 1.27 1.27)
-				)
-			)
-		)
-		(property "Description" "10V 4.7uF X5R ±10% 0402 Multilayer Ceramic Capacitors MLCC - SMD/SMT ROHS"
+		(property "Datasheet" ""
 			(at 265.43 30.48 0)
 			(hide yes)
@@
 			)
 		)
-		(property "LCSC" "C368809"
+		(property "Description" ""
 			(at 265.43 30.48 0)
 			(hide yes)
@@
 			)
 		)
-		(property "Manufacturer" "Samsung Electro-Mechanics"
+		(property "LCSC" "C23733"
 			(at 265.43 30.48 0)
 			(hide yes)
@@
 			)
 		)
-		(property "Datasheet" "https://www.lcsc.com/datasheet/lcsc_datasheet_2410121857_Murata-Electronics-GRM1555C1H100JA01D_C76946.pdf"
+		(property "Datasheet" ""
 			(at 372.11 223.52 0)
 			(hide yes)
@@
 			)
 		)
-		(property "Description" "50V 10pF C0G ±5% 0402 Multilayer Ceramic Capacitors MLCC - SMD/SMT ROHS"
+		(property "Description" ""
 			(at 372.11 223.52 0)
 			(hide yes)
@@
 			)
 		)
-		(property "LCSC" "C76946"
+		(property "LCSC" "C32949"
 			(at 372.11 223.52 0)
 			(hide yes)
@@
 			)
 		)
-		(property "Manufacturer" "Murata Electronics"
+		(property "Manufacturer" ""
 			(at 372.11 223.52 0)
 			(hide yes)
@@
 		(in_pos_files yes)
 		(dnp no)
-		(fields_autoplaced yes)
 		(property "Reference" "R9"
 			(at 71.12 35.56 90)
@@
 			)
 		)
-		(property "Value" "22"
-			(at 71.12 38.1 90)
+		(property "Value" "22R"
+			(at 71.374 38.862 90)
 			(show_name no)
 			(do_not_autoplace no)
@@
 			)
 		)
-		(property "Datasheet" "https://www.lcsc.com/datasheet/lcsc_datasheet_2410121857_Murata-Electronics-GRM1555C1H100JA01D_C76946.pdf"
+		(property "Datasheet" ""
 			(at 397.51 223.52 0)
 			(hide yes)
@@
 			)
 		)
-		(property "Description" "50V 10pF C0G ±5% 0402 Multilayer Ceramic Capacitors MLCC - SMD/SMT ROHS"
+		(property "Description" ""
 			(at 397.51 223.52 0)
 			(hide yes)
@@
 			)
 		)
-		(property "LCSC" "C76946"
+		(property "LCSC" "C32949"
 			(at 397.51 223.52 0)
 			(hide yes)
@@
 			)
 		)
-		(property "Manufacturer" "Murata Electronics"
+		(property "Manufacturer" ""
 			(at 397.51 223.52 0)
 			(hide yes)
@@
 			)
 		)
-		(property "Value" "22"
-			(at 34.29 38.1 90)
+		(property "Value" "22R"
+			(at 34.29 37.338 90)
 			(show_name no)
 			(do_not_autoplace no)
@@
 			)
 		)
-		(property "Value" "22"
+		(property "Value" "22R"
 			(at 34.29 26.924 90)
 			(show_name no)
@@
 			)
 		)
-		(property "Datasheet" "https://www.lcsc.com/datasheet/lcsc_datasheet_2304140030_YAGEO-CC0402KRX7R9BB103_C60133.pdf"
+		(property "Datasheet" ""
 			(at 391.16 30.48 0)
 			(hide yes)
@@
 			)
 		)
-		(property "Description" "50V 10nF X7R ±10% 0402 Multilayer Ceramic Capacitors MLCC - SMD/SMT ROHS"
+		(property "Description" ""
 			(at 391.16 30.48 0)
 			(hide yes)
@@
 			)
 		)
-		(property "LCSC" "C60133"
+		(property "LCSC" "C15195"
 			(at 391.16 30.48 0)
 			(hide yes)
@@
 			)
 		)
-		(property "Manufacturer" "YAGEO"
+		(property "Manufacturer" ""
 			(at 391.16 30.48 0)
 			(hide yes)
@@
 			)
 		)
-		(property "Value" "TS342A2P"
+		(property "Value" ""
 			(at 233.553 98.2222 90)
 			(show_name no)
@@
 			)
 		)
-		(property "Footprint" "Button_Switch_SMD:SW_Push_SPST_NO_Alps_SKRK"
+		(property "Footprint" "Button_Switch_SMD:SW_SPST_TS-1088-xR020"
 			(at 232.41 96.52 0)
 			(hide yes)
@@
 			)
 		)
-		(property "LCSC" "C5373431"
+		(property "LCSC" "C720477"
 			(at 232.41 96.52 0)
 			(hide yes)
@@
 			)
 		)
-		(property "Value" "22"
-			(at 39.37 45.72 90)
+		(property "Value" "22R"
+			(at 39.37 44.958 90)
 			(show_name no)
 			(do_not_autoplace no)
@@
 			)
 		)
-		(property "Value" "TS342A2P"
+		(property "Value" ""
 			(at 227.203 63.9322 90)
 			(show_name no)
@@
 			)
 		)
-		(property "Footprint" "Button_Switch_SMD:SW_Push_SPST_NO_Alps_SKRK"
+		(property "Footprint" "Button_Switch_SMD:SW_SPST_TS-1088-xR020"
 			(at 226.06 62.23 0)
 			(hide yes)
@@
 			)
 		)
-		(property "LCSC" "C5373431"
+		(property "LCSC" "C720477"
 			(at 226.06 62.23 0)
 			(hide yes)
