File: rapid_power_module.kicad_sch (KiCad schematic)
At the start: 26 parts, among them J1 Conn_02x04_Top_Bottom, J2 Molex MicroFit 2x2, J3 Conn_02x04_Top_Bottom, J4 Molex MicroFit 2x2, J5 Molex MicroFit 2x2, J6 Molex MicroFit 2x2, J7 Molex MicroFit 2x2

Commit message: added missing footprints and validated all lcsc numbers; started pcb-layouting
Parts:
- F3, J1, J3: LCSC (none) -> x; now not fitted
- FB2: LCSC (none) -> C304323; LCSC# C304323 -> (none)
- H1, H2, H3, H4: DigiKey# N/A -> (none); LCSC (none) -> x; LCSC# N/A -> (none); Manufacturer N/A -> (none); Part# N/A -> (none)
- J5: now not fitted
- J6, J7: LCSC (none) -> C122413; LCSC# C122413 -> (none); Manufacturer MOLEX -> (none); now not fitted
Connections:
- net BAL_GND renamed GND
Other:
- sheet Balancer ports: added BAT-; removed none
Changed lines of the file:
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@@
 	(text "Arming Connector"
 		(exclude_from_sim no)
-		(at 38.1 80.01 0)
+		(at 35.814 80.518 0)
 		(effects
 			(font
@@
 	)
 	(junction
-		(at 369.57 34.29)
-		(diameter 0)
-		(color 0 0 0 0)
-	)
-	(junction
 		(at 36.83 45.72)
 		(diameter 0)
@@
 	(wire
 		(pts
-			(xy 369.57 34.29) (xy 379.73 34.29)
-		)
-		(stroke
-			(width 0)
-			(type default)
-		)
-	)
-	(wire
-		(pts
 			(xy 83.82 135.89) (xy 85.09 135.89)
 		)
@@
 	(wire
 		(pts
-			(xy 379.73 34.29) (xy 379.73 36.83)
-		)
-		(stroke
-			(width 0)
-			(type default)
-		)
-	)
-	(wire
-		(pts
 			(xy 33.02 43.18) (xy 36.83 43.18)
 		)
@@
 	(wire
 		(pts
+			(xy 288.29 151.13) (xy 294.64 151.13)
+		)
+		(stroke
+			(width 0)
+			(type default)
+		)
+	)
+	(wire
+		(pts
 			(xy 50.8 45.72) (xy 54.61 45.72)
 		)
@@
 			)
 		)
-		(property "Manufacturer" "N/A"
+		(property "LCSC" "x"
 			(at 109.22 49.53 0)
 			(effects
@@
 			)
 		)
-		(property "Part#" "N/A"
-			(at 109.22 49.53 0)
+		(pin "1"
+		)
+		(instances
+			(project "frodo_power_module"
+				(path "/afc8cbd3-9ea8-40a2-afae-ed6bd0fe7e6e"
+					(reference "H2")
+					(unit 1)
+				)
+			)
+		)
+	)
+	(symbol
+		(lib_name "GND_1")
+		(lib_id "power:GND")
+		(at 288.29 151.13 270)
+		(unit 1)
+		(exclude_from_sim no)
+		(in_bom yes)
+		(on_board yes)
+		(dnp no)
+		(property "Reference" "#PWR05"
+			(at 281.94 151.13 0)
 			(effects
 				(font
@@
 			)
 		)
-		(property "DigiKey#" "N/A"
-			(at 109.22 49.53 0)
+		(property "Value" "GND"
+			(at 284.226 151.13 0)
+			(effects
+				(font
+					(size 1.27 1.27)
+				)
+			)
+		)
+		(property "Footprint" ""
+			(at 288.29 151.13 0)
 			(effects
 				(font
@@
 			)
 		)
-		(property "LCSC#" "N/A"
-			(at 109.22 49.53 0)
+		(property "Datasheet" ""
+			(at 288.29 151.13 0)
+			(effects
+				(font
+					(size 1.27 1.27)
+				)
+				(hide yes)
+			)
+		)
+		(property "Description" "Power symbol creates a global label with name \"GND\" , ground"
+			(at 288.29 151.13 0)
 			(effects
 				(font
@@
 		)
 		(instances
-			(project "frodo_power_module"
+			(project "rapid_power_module"
 				(path "/afc8cbd3-9ea8-40a2-afae-ed6bd0fe7e6e"
-					(reference "H2")
+					(reference "#PWR05")
 					(unit 1)
 				)
@@
 		(in_bom yes)
 		(on_board yes)
-		(dnp no)
+		(dnp yes)
 		(property "Reference" "J5"
 			(at 20.32 93.472 90)
@@
 		(in_bom yes)
 		(on_board yes)
-		(dnp no)
+		(dnp yes)
 		(property "Reference" "J6"
 			(at 20.828 133.35 0)
@@
 			)
 		)
-		(property "LCSC#" "C122413"
-			(at 22.86 134.62 0)
-			(effects
-				(font
-					(size 1.27 1.27)
-				)
-				(hide yes)
-			)
-		)
-		(property "Manufacturer" "MOLEX"
+		(property "LCSC" "C122413"
 			(at 22.86 134.62 0)
 			(effects
@@
 			)
 		)
-		(property "Manufacturer" "N/A"
-			(at 109.22 55.88 0)
-			(effects
-				(font
-					(size 1.27 1.27)
-				)
-				(hide yes)
-			)
-		)
-		(property "Part#" "N/A"
-			(at 109.22 55.88 0)
-			(effects
-				(font
-					(size 1.27 1.27)
-				)
-				(hide yes)
-			)
-		)
-		(property "DigiKey#" "N/A"
-			(at 109.22 55.88 0)
-			(effects
-				(font
-					(size 1.27 1.27)
-				)
-				(hide yes)
-			)
-		)
-		(property "LCSC#" "N/A"
+		(property "LCSC" "x"
 			(at 109.22 55.88 0)
 			(effects
@@
 		(in_bom yes)
 		(on_board yes)
-		(dnp no)
+		(dnp yes)
 		(property "Reference" "J7"
 			(at 20.828 154.94 0)
@@
 			)
 		)
-		(property "LCSC#" "C122413"
-			(at 22.86 156.21 0)
-			(effects
-				(font
-					(size 1.27 1.27)
-				)
-				(hide yes)
-			)
-		)
-		(property "Manufacturer" "MOLEX"
+		(property "LCSC" "C122413"
 			(at 22.86 156.21 0)
 			(effects
@@
 			)
 		)
-		(property "Manufacturer" "N/A"
-			(at 109.22 43.18 0)
-			(effects
-				(font
-					(size 1.27 1.27)
-				)
-				(hide yes)
-			)
-		)
-		(property "Part#" "N/A"
-			(at 109.22 43.18 0)
-			(effects
-				(font
-					(size 1.27 1.27)
-				)
-				(hide yes)
-			)
-		)
-		(property "DigiKey#" "N/A"
-			(at 109.22 43.18 0)
-			(effects
-				(font
-					(size 1.27 1.27)
-				)
-				(hide yes)
-			)
-		)
-		(property "LCSC#" "N/A"
+		(property "LCSC" "x"
 			(at 109.22 43.18 0)
 			(effects
@@
 		(in_bom yes)
 		(on_board yes)
-		(dnp no)
+		(dnp yes)
 		(property "Reference" "J1"
 			(at 44.45 40.386 0)
@@
 			)
 		)
+		(property "LCSC" "x"
+			(at 43.18 45.72 0)
+			(effects
+				(font
+					(size 1.27 1.27)
+				)
+				(hide yes)
+			)
+		)
 		(pin "6"
 		)
@@
 		(in_bom yes)
 		(on_board yes)
-		(dnp no)
+		(dnp yes)
 		(property "Reference" "F3"
 			(at 237.236 152.146 90)
@@
 			)
 		)
+		(property "LCSC" "x"
+			(at 237.49 149.86 90)
+			(effects
+				(font
+					(size 1.27 1.27)
+				)
+				(hide yes)
+			)
+		)
 		(pin "1"
 		)
@@
 			)
 		)
-		(property "LCSC#" "C304323"
+		(property "LCSC" "C304323"
 			(at 57.15 93.98 0)
 			(effects
@@
 	(symbol
 		(lib_id "power:GND")
-		(at 379.73 36.83 0)
-		(unit 1)
-		(exclude_from_sim no)
-		(in_bom yes)
-		(on_board yes)
-		(dnp no)
-		(property "Reference" "#PWR05"
-			(at 379.73 43.18 0)
-			(effects
-				(font
-					(size 1.27 1.27)
-				)
-				(hide yes)
-			)
-		)
-		(property "Value" "BAL_GND"
-			(at 379.73 40.894 0)
-			(effects
-				(font
-					(size 1.27 1.27)
-				)
-			)
-		)
-		(property "Footprint" ""
-			(at 379.73 36.83 0)
-			(effects
-				(font
-					(size 1.27 1.27)
-				)
-				(hide yes)
-			)
-		)
-		(property "Datasheet" ""
-			(at 379.73 36.83 0)
-			(effects
-				(font
-					(size 1.27 1.27)
-				)
-				(hide yes)
-			)
-		)
-		(property "Description" "Power symbol creates a global label with name \"GND\" , ground"
-			(at 379.73 36.83 0)
-			(effects
-				(font
-					(size 1.27 1.27)
-				)
-				(hide yes)
-			)
-		)
-		(pin "1"
-		)
-		(instances
-			(project "rapid_power_module"
-				(path "/afc8cbd3-9ea8-40a2-afae-ed6bd0fe7e6e"
-					(reference "#PWR05")
-					(unit 1)
-				)
-			)
-		)
-	)
-	(symbol
-		(lib_id "power:GND")
 		(at 243.84 138.43 0)
 		(unit 1)
@@
 		(in_bom yes)
 		(on_board yes)
-		(dnp no)
+		(dnp yes)
 		(property "Reference" "J3"
 			(at 44.45 55.626 0)
@@
 			)
 		)
+		(property "LCSC" "x"
+			(at 43.18 60.96 0)
+			(effects
+				(font
+					(size 1.27 1.27)
+				)
+				(hide yes)
+			)
+		)
 		(pin "6"
 		)
@@
 			)
 		)
-		(property "Manufacturer" "N/A"
-			(at 109.22 62.23 0)
-			(effects
-				(font
-					(size 1.27 1.27)
-				)
-				(hide yes)
-			)
-		)
-		(property "Part#" "N/A"
-			(at 109.22 62.23 0)
-			(effects
-				(font
-					(size 1.27 1.27)
-				)
-				(hide yes)
-			)
-		)
-		(property "DigiKey#" "N/A"
-			(at 109.22 62.23 0)
-			(effects
-				(font
-					(size 1.27 1.27)
-				)
-				(hide yes)
-			)
-		)
-		(property "LCSC#" "N/A"
+		(property "LCSC" "x"
 			(at 109.22 62.23 0)
 			(effects
@@
 			(effects
 				(font
+					(size 1.27 1.27)
+				)
+				(justify left)
+			)
+		)
+		(pin "BAT-" bidirectional
+			(at 294.64 151.13 180)
+			(effects
+				(font

Commit message: started routing Please enter the commit message for your changes. Lines starting
Other:
- note added: "Main Switch"
- note removed: "Arming Connector"
Changed lines of the file:
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@@
 		)
 	)
-	(text "Arming Connector"
+	(text "Main Switch"
 		(exclude_from_sim no)
-		(at 35.814 80.518 0)
+		(at 29.972 80.518 0)
 		(effects
 			(font
