File: charger.kicad_sch (KiCad schematic)
At the start: 34 parts, among them U6 BQ25798RQMR

Commit message: edited do not place
Parts:
- TH1: now not fitted
Changed lines of the file:
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@@
 		(on_board yes)
 		(in_pos_files yes)
-		(dnp no)
+		(dnp yes)
 		(fields_autoplaced yes)
 		(property "Reference" "TH1"

Commit message: last changes (components) for ordering
Parts:
- C37: LCSC C368809 -> C23733; Manufacturer Samsung Electro-Mechanics -> (none)
- R29: LCSC C4190 -> C25879
Changed lines of the file:
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@@
 			)
 		)
-		(property "Datasheet" "https://www.lcsc.com/datasheet/lcsc_datasheet_2304140030_Samsung-Electro-Mechanics-CL05A475KP5NRNC_C368809.pdf"
+		(property "Datasheet" ""
 			(at 106.68 86.36 0)
 			(hide yes)
@@
 			)
 		)
-		(property "Description" "10V 4.7uF X5R ±10% 0402 Multilayer Ceramic Capacitors MLCC - SMD/SMT ROHS"
+		(property "Description" ""
 			(at 106.68 86.36 0)
 			(hide yes)
@@
 			)
 		)
-		(property "LCSC" "C368809"
+		(property "LCSC" "C23733"
 			(at 106.68 86.36 0)
 			(hide yes)
@@
 			)
 		)
-		(property "Manufacturer" "Samsung Electro-Mechanics"
+		(property "Manufacturer" ""
 			(at 106.68 86.36 0)
 			(hide yes)
@@
 			)
 		)
-		(property "LCSC" "C4190"
+		(property "LCSC" "C25879"
 			(at 175.26 105.41 90)
 			(hide yes)
